Commit message: 导航实现

File: src/R1/urdf/R1.urdf (robot description, URDF)
Before this commit: robot R1, 10 links, 9 joints
Joints:
- joint J2: axis 0 -1 0 -> 0 1 0
- joint J3: axis 0 -1 0 -> 0 1 0
- joint J4: axis 0 1 0 -> 0 -1 0
- joint base_footprint_joint: origin xyz=0 0 0.04075 rpy=0 0 0 -> xyz=0 0 0.04075 rpy=0 0 3.14159265359
- joint camera_joint: origin xyz=-0.26 0 0.24 rpy=0 0 3.14159265359 -> xyz=-0.30 0 0.28 rpy=0 0 3.14159265359
- joint laser_joint: origin xyz=-0.24 0 0.31 rpy=0 0 3.14159265359 -> xyz=-0.34 0 0.36 rpy=0 0 3.14159265359

Commit message: 避障实现

File: src/R1/urdf/R1.urdf (robot description, URDF)
Before this commit: robot R1, 10 links, 9 joints
Links:
- link base_link: geometry collision box size=0.40 0.03 0.02; collision box size=0.40 0.03 0.02
Joints:
- joint J1: axis 0 -1 0 -> 0 1 0; origin xyz=-0.220127909860013 -0.142085316479216 0.0 rpy=0 0 0 -> xyz=0.220127909860013 0.142085316479216 0.0 rpy=0 0 0
- joint J2: axis 0 1 0 -> 0 -1 0; origin xyz=-0.220127909860013 0.122535316479216 0.0 rpy=0 0 0 -> xyz=0.220127909860013 -0.122535316479216 0.0 rpy=0 0 0
- joint J3: axis 0 1 0 -> 0 -1 0; origin xyz=0.19879978611665 0.122535316479219 0.0 rpy=0 0 0 -> xyz=-0.19879978611665 -0.122535316479219 0.0 rpy=0 0 0
- joint J4: axis 0 -1 0 -> 0 1 0; origin xyz=0.19879978611665 -0.119285316479219 0.0 rpy=0 0 0 -> xyz=-0.19879978611665 0.119285316479219 0.0 rpy=0 0 0
- joint base_footprint_joint: origin xyz=0 0 0.04075 rpy=0 0 3.14159265359 -> xyz=0 0 0.04075 rpy=0 0 0
- joint camera_joint: origin xyz=-0.30 0 0.28 rpy=0 0 3.14159265359 -> xyz=0.30 0 0.28 rpy=0 0 0
- joint imu_joint: origin xyz=-0.02 0 0.22 rpy=0 0 0 -> xyz=0.02 0 0.22 rpy=0 0 0
- joint laser_joint: origin xyz=-0.34 0 0.36 rpy=0 0 3.14159265359 -> xyz=0.34 0 0.36 rpy=0 0 0

File: src/R1/urdf/R1_rviz.urdf (robot description, URDF)
Before this commit: robot R1_rviz, 10 links, 9 joints
Joints:
- joint J1: axis 0 -1 0 -> 0 1 0; origin xyz=-0.220127909860013 -0.142085316479216 0.0 rpy=0 0 0 -> xyz=0.220127909860013 0.142085316479216 0.0 rpy=0 0 0
- joint J2: axis 0 1 0 -> 0 -1 0; origin xyz=-0.220127909860013 0.122535316479216 0.0 rpy=0 0 0 -> xyz=0.220127909860013 -0.122535316479216 0.0 rpy=0 0 0
- joint J3: axis 0 1 0 -> 0 -1 0; origin xyz=0.19879978611665 0.122535316479219 0.0 rpy=0 0 0 -> xyz=-0.19879978611665 -0.122535316479219 0.0 rpy=0 0 0
- joint J4: axis 0 -1 0 -> 0 1 0; origin xyz=0.19879978611665 -0.119285316479219 0.0 rpy=0 0 0 -> xyz=-0.19879978611665 0.119285316479219 0.0 rpy=0 0 0
- joint base_footprint_joint: origin xyz=0 0 0.04075 rpy=0 0 3.14159265359 -> xyz=0 0 0.04075 rpy=0 0 0
- joint camera_joint: origin xyz=-0.30 0 0.28 rpy=0 0 3.14159265359 -> xyz=0.30 0 0.28 rpy=0 0 0
- joint imu_joint: origin xyz=-0.02 0 0.22 rpy=0 0 0 -> xyz=0.02 0 0.22 rpy=0 0 0
- joint laser_joint: origin xyz=-0.34 0 0.36 rpy=0 0 3.14159265359 -> xyz=0.34 0 0.36 rpy=0 0 0

Commit message: 修复前轮脱离情况

File: src/R1/urdf/R1.urdf (robot description, URDF)
Before this commit: robot R1, 10 links, 9 joints
Joints:
- joint J1: origin xyz=0.220127909860013 0.142085316479216 0.0 rpy=0 0 0 -> xyz=0.220127909860013 0.122535316479216 0.0 rpy=0 0 0
- joint J2: origin xyz=0.220127909860013 -0.122535316479216 0.0 rpy=0 0 0 -> xyz=0.220127909860013 -0.142085316479216 0.0 rpy=0 0 0

File: src/R1/urdf/R1_rviz.urdf (robot description, URDF)
Before this commit: robot R1_rviz, 10 links, 9 joints
Joints:
- joint J1: origin xyz=0.220127909860013 0.142085316479216 0.0 rpy=0 0 0 -> xyz=0.220127909860013 0.122535316479216 0.0 rpy=0 0 0
- joint J2: origin xyz=0.220127909860013 -0.122535316479216 0.0 rpy=0 0 0 -> xyz=0.220127909860013 -0.142085316479216 0.0 rpy=0 0 0

Commit message: 完善前驱阿克曼自主导航仿真链路
本次提交围绕 500kg 前轮驱动 Ackermann 小车的自主导航效果做全链路修复。主要内容包括：

1. 接入 ackermann_steering_controller，新增 ros_controllers.yaml，并在 Gazebo 启动链路中加载 ros_control 控制器。

2. 将 URDF 调整为前轮转向、前轮驱动结构，更新质量/惯量、轮胎接触参数、canonical body 和 ground truth 绑定，减少 root inertia 与仿真位姿问题。

3. 新增 cmd_vel 到 Ackermann 转角的适配器，把 move_base 输出的 yaw rate 转成 steering angle，并显式忽略横向速度。

4. 新增 Gazebo Ackermann effort bridge，用 ground truth 速度闭环施加驱动力和转向力，改善前驱重车在仿真中的起步、制动和弧线跟踪。

5. 改造 odom_sanitizer，让仿真默认使用平面化 ground truth odom 发布 odom -> base_footprint，避免原控制器轮速里程计与真实位姿严重不一致。

6. 重调 DWA 障碍导航参数，限制横向速度和不可实现的原地旋转曲率，按阿克曼最小转弯半径改成前进弧线规划。

7. 更新导航、障碍测试、sim bringup、地图和恢复行为配置，禁用旋转恢复，保留 costmap 清理恢复。

验证：catkin_make --pkg r1 通过；Python 脚本编译通过；launch/URDF XML 检查通过；URDF 到 SDF 转换通过；nav_obstacle_test 中目标 (2.94, -1.96) 到达成功，move_base 返回 Goal reached。

File: src/R1/urdf/R1.urdf (robot description, URDF)
Before this commit: robot R1, 10 links, 9 joints
Links:
- added link front_drive_wheel_link, mass 12.0; collision cylinder length=0.040 radius=0.04075
- added link front_steer_link, mass 5.0
- link Empty_Link1: mass 0.102007563940439 -> 1.0; geometry visual mesh filename=package://r1/meshes/Empty_Link1.STL
- link Empty_Link2: mass 0.102007476255524 -> 1.0; geometry visual mesh filename=package://r1/meshes/Empty_Link2.STL
- link Empty_Link3: mass 0.130385211409052 -> 6.0
- link Empty_Link4: mass 0.130386181839137 -> 6.0
- link base_link: mass 38.0603057004842 -> 470.0
Joints:
- added joint front_drive_wheel_joint: type continuous, parent front_steer_link, child front_drive_wheel_link, origin xyz=0 0 0 rpy=0 0 0, axis 0 1 0, limit effort=1200 velocity=30
- added joint front_steer_joint: type revolute, parent base_link, child front_steer_link, origin xyz=0.220127909860013 -0.009775 0.0 rpy=0 0 0, axis 0 0 1, limit lower=-0.6 upper=0.6 effort=5000 velocity=1.5
- joint J1: limit effort=20 velocity=20 -> effort=200 velocity=20; origin xyz=0.220127909860013 0.122535316479216 0.0 rpy=0 0 0 -> xyz=0 0.132310316479216 0.0 rpy=0 0 0; parent base_link -> front_steer_link
- joint J2: axis 0 -1 0 -> 0 1 0; limit effort=20 velocity=20 -> effort=200 velocity=20; origin xyz=0.220127909860013 -0.142085316479216 0.0 rpy=0 0 0 -> xyz=0 -0.132310316479216 0.0 rpy=0 0 0; parent base_link -> front_steer_link
- joint J3: axis 0 -1 0 -> 0 1 0; limit effort=20 velocity=20 -> effort=200 velocity=20
- joint J4: limit effort=20 velocity=20 -> effort=200 velocity=20
