Commit message: 健全teb参数，并加上pid控制

File: zebrat/urdf/R1.urdf (robot description, URDF)
Before this commit: robot R1, 11 links, 10 joints
Joints:
- joint front_left_steering_joint: origin xyz=0.220127909860013 0.142085316479216 0.04075 rpy=0 0 0 -> xyz=0.220127909860013 0.132310316479216 0.04075 rpy=0 0 0
- joint front_right_steering_joint: origin xyz=0.220127909860013 -0.122535316479216 0.04075 rpy=0 0 0 -> xyz=0.220127909860013 -0.132310316479216 0.04075 rpy=0 0 0
- joint rear_left_wheel_joint: origin xyz=-0.19879978611665 0.119285316479219 0.0 rpy=0 0 0 -> xyz=-0.19879978611665 0.120910316479219 0.0 rpy=0 0 0
- joint rear_right_wheel_joint: origin xyz=-0.19879978611665 -0.122535316479219 0.0 rpy=0 0 0 -> xyz=-0.19879978611665 -0.120910316479219 0.0 rpy=0 0 0

File: zebrat/urdf/R1_rviz.urdf (robot description, URDF)
Before this commit: robot R1_rviz, 12 links, 11 joints
Joints:
- joint front_left_steering_joint: origin xyz=0.220127909860013 0.142085316479216 0.04075 rpy=0 0 0 -> xyz=0.220127909860013 0.132310316479216 0.04075 rpy=0 0 0
- joint front_right_steering_joint: origin xyz=0.220127909860013 -0.122535316479216 0.04075 rpy=0 0 0 -> xyz=0.220127909860013 -0.132310316479216 0.04075 rpy=0 0 0
- joint rear_left_wheel_joint: origin xyz=-0.19879978611665 0.119285316479219 0.0 rpy=0 0 0 -> xyz=-0.19879978611665 0.120910316479219 0.0 rpy=0 0 0
- joint rear_right_wheel_joint: origin xyz=-0.19879978611665 -0.122535316479219 0.0 rpy=0 0 0 -> xyz=-0.19879978611665 -0.120910316479219 0.0 rpy=0 0 0

Commit message: 稳定 R1 TEB 阿克曼转向

File: zebrat/urdf/R1.urdf (robot description, URDF)
Before this commit: robot R1, 11 links, 10 joints
Joints:
- joint camera_joint: origin xyz=0.30 0 0.28 rpy=0 0 0 -> xyz=0.49879978611665 0 0.28 rpy=0 0 0
- joint front_left_steering_joint: origin xyz=0.220127909860013 0.132310316479216 0.04075 rpy=0 0 0 -> xyz=0.418927695976663 0.132310316479216 0.04075 rpy=0 0 0
- joint front_right_steering_joint: origin xyz=0.220127909860013 -0.132310316479216 0.04075 rpy=0 0 0 -> xyz=0.418927695976663 -0.132310316479216 0.04075 rpy=0 0 0
- joint imu_joint: origin xyz=0.02 0 0.22 rpy=0 0 0 -> xyz=0.21879978611665 0 0.22 rpy=0 0 0
- joint laser_joint: origin xyz=0.34 0 0.36 rpy=0 0 0 -> xyz=0.53879978611665 0 0.36 rpy=0 0 0
- joint rear_left_wheel_joint: origin xyz=-0.19879978611665 0.120910316479219 0.0 rpy=0 0 0 -> xyz=0.0 0.120910316479219 0.0 rpy=0 0 0
- joint rear_right_wheel_joint: origin xyz=-0.19879978611665 -0.120910316479219 0.0 rpy=0 0 0 -> xyz=0.0 -0.120910316479219 0.0 rpy=0 0 0

File: zebrat/urdf/R1_rviz.urdf (robot description, URDF)
Before this commit: robot R1_rviz, 12 links, 11 joints
Joints:
- joint camera_joint: origin xyz=0.30 0 0.28 rpy=0 0 0 -> xyz=0.49879978611665 0 0.28 rpy=0 0 0
- joint front_left_steering_joint: origin xyz=0.220127909860013 0.132310316479216 0.04075 rpy=0 0 0 -> xyz=0.418927695976663 0.132310316479216 0.04075 rpy=0 0 0
- joint front_right_steering_joint: origin xyz=0.220127909860013 -0.132310316479216 0.04075 rpy=0 0 0 -> xyz=0.418927695976663 -0.132310316479216 0.04075 rpy=0 0 0
- joint imu_joint: origin xyz=0.02 0 0.22 rpy=0 0 0 -> xyz=0.21879978611665 0 0.22 rpy=0 0 0
- joint laser_joint: origin xyz=0.34 0 0.36 rpy=0 0 0 -> xyz=0.53879978611665 0 0.36 rpy=0 0 0
- joint rear_left_wheel_joint: origin xyz=-0.19879978611665 0.120910316479219 0.0 rpy=0 0 0 -> xyz=0.0 0.120910316479219 0.0 rpy=0 0 0
- joint rear_right_wheel_joint: origin xyz=-0.19879978611665 -0.120910316479219 0.0 rpy=0 0 0 -> xyz=0.0 -0.120910316479219 0.0 rpy=0 0 0
